Commit message: With SLAM

File: description/lidar.xacro (robot description, xacro)
@@ -26,5 +26,5 @@
         <sensor name="laser" type="ray">
             <pose> 0 0 0 0 0 0</pose>
-            <visualize>true</visualize>
+            <visualize>false</visualize>
             <update_rate>10</update_rate>
             <ray>

File: description/robot.urdf.xacro (robot description, xacro)
@@ -1,7 +1,14 @@
 <?xml version="1.0"?>
 <robot xmlns:xacro="http://www.ros.org/wiki/xacro"  name="robot">
+    <xacro:arg name="use_ros2_control" default="true" />
     <xacro:include filename="robot_core.xacro" />
-    <!-- <xacro:include filename="gazebo_control.xacro" /> -->
-     <xacro:include filename="ros2_control.xacro" />
+    <!-- <xacro:include filename="ros2_control.xacro" /> -->
+    <!-- <xacro:include filename="gazebo_control.xacro"/> -->
+    <xacro:if value="$(arg use_ros2_control)">
+        <xacro:include filename="ros2_control.xacro" />
+    </xacro:if>
+    <xacro:unless value="$(arg use_ros2_control)">
+        <xacro:include filename="gazebo_control.xacro" />
+    </xacro:unless>
     <xacro:include filename="lidar.xacro" />
     <xacro:include filename="camera.xacro" />

File: description/robot_core.xacro (robot description, xacro)
@@ -19,4 +19,12 @@
     <!-- BASE LINK -->
     <link name="base_link">
+    </link>
+    <!-- BASE_FOOTPRINT LINK-->
+    <joint name="base_footprint_joint" type="fixed">
+        <parent link="base_link" />
+        <child link="base_footprint" />
+        <origin xyz="0 0 0" rpy="0 0 0" />
+    </joint>
+    <link name="base_footprint">
     </link>
     <!-- CHASSIS LINK -->
@@ -63,5 +71,5 @@
     <collision>
         <geometry>
-            <cylinder length="0.04" radius="0.05" />
+            <sphere radius="0.05" />
         </geometry>
     </collision>
@@ -89,5 +97,5 @@
     <collision>
         <geometry>
-            <cylinder length="0.04" radius="0.05" />
+            <sphere radius="0.05" />
         </geometry>
     </collision>

File: description/ros2_control.xacro (robot description, xacro)
@@ -1,4 +1,32 @@
 <?xml version="1.0"?>
 <robot xmlns:xacro="http://www.ros.org/wiki/xacro">
+    <ros2_control name="RealRobot" type="system">
+        <hardware>
+            <plugin>diffdrive_arduino/DiffDriveArduino</plugin>
+            <param name ='left_wheel_name'>left_wheel_joint</param>
+            <param name ='right_wheel_name'>right_wheel_joint</param>
+            <param name ='loop_rate'>30</param>
+            <param name ='devices'>/dev/ttyUSB0</param>
+            <param name ='baud_rate'>57600</param>
+            <param name ='timeout'>1000</param>
+            <param name ='end_counts_per_rev'>3450</param>
+        </hardware>
+        <joint name="left_wheel_joint">
+            <command_interface name="velocity">
+                <param name="min">-10</param>
+                <param name="max">10</param>
+            </command_interface>
+            <state_interface name="position" />
+            <state_interface name="velocity" />
+        </joint>
+        <joint name="right_wheel_joint">
+            <command_interface name="velocity">
+                <param name="min">-10</param>
+                <param name="max">10</param>
+            </command_interface>
+            <state_interface name="velocity" />
+            <state_interface name="position" />
+        </joint>
+    </ros2_control>
     <ros2_control name="GazeboSystem" type="system">
         <hardware>
